Commit message: 2026.03.15

File: ros2_ws/src/robot_control/urdf/simple_robot_gazebo.urdf (robot description, URDF)
Before this commit: robot two_wheel_robot, 4 links, 3 joints
Links:
- link base_link: mass 2.0 -> 4.0
- link caster_wheel: mass 0.1 -> 0.2
- link left_wheel: mass 0.3 -> 0.5
- link right_wheel: mass 0.3 -> 0.5
Joints:
- joint caster_joint: origin xyz=-0.12 0 -0.05 -> xyz=-0.12 0 0.015 rpy=0 0 0
- joint left_wheel_joint: axis 0 1 0 -> 1 0 0; limit (none) -> effort=10 velocity=10; origin xyz=0 0.11 -0.05 -> xyz=0 0.11 0.05 rpy=0 0 0
- joint right_wheel_joint: axis 0 1 0 -> 1 0 0; limit (none) -> effort=10 velocity=10; origin xyz=0 -0.11 -0.05 -> xyz=0 -0.11 0.05 rpy=0 0 0

Commit message: 2026.03.18

File: ros2_ws/src/robot_control/urdf/simple_robot_gazebo.urdf (robot description, URDF)
Before this commit: robot two_wheel_robot, 4 links, 3 joints
Joints:
- joint caster_joint: origin xyz=-0.12 0 0.015 rpy=0 0 0 -> xyz=-0.12 0 0.03 rpy=0 0 0
- joint left_wheel_joint: axis 1 0 0 -> 0 1 0; origin xyz=0 0.11 0.05 rpy=0 0 0 -> xyz=0.03 0.11 0.05 rpy=0 0 0
- joint right_wheel_joint: axis 1 0 0 -> 0 1 0; origin xyz=0 -0.11 0.05 rpy=0 0 0 -> xyz=0.03 -0.11 0.05 rpy=0 0 0

Commit message: Add LiDAR scan support and headless launch option

File: ros2_ws/src/robot_control/urdf/simple_robot_gazebo.urdf (robot description, URDF)
Before this commit: robot two_wheel_robot, 4 links, 3 joints
Links:
- added link lidar_link, mass 0.1; collision cylinder length=0.04 radius=0.04; visual cylinder length=0.04 radius=0.04
Joints:
- added joint lidar_joint: type fixed, parent base_link, child lidar_link, origin xyz=0.10 0 0.18 rpy=0 0 0
